File: Serberus.kicad_pcb (KiCad board)
At the start: 4 copper layers, 65 x 61 mm, 108 parts, among them J1 USB_C_Receptacle_USB2.0, J2 UART 1,3,4, J3 SWD/JTAG2, J4 LA, J5 SPI, J6 CORTEX, J7 I2C, J8 iCE40, J9 V_Merge, Q1 BSH103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

Commit message: Changed to V1.1
Parts:
- C25: value NF -> DNP
- C28: value .1u -> 100n
- R15: value 2.2k -> 2k2
- moved C1 7.52 mm to (126.2, 76.6), turned to 90 degrees
- moved C2 7.44 mm to (129.6, 73.6)
- moved U1 7.17 mm to (128.6, 76.0)
- moved C4 4.75 mm to (130.0, 80.4), turned to -90 degrees
- moved R11 4.02 mm to (141.4, 88.2), turned to 180 degrees
- moved C3 3.98 mm to (125.0, 81.4), turned to 90 degrees
- moved C7 3.50 mm to (125.8, 83.2), turned to 180 degrees
- moved R21 2.30 mm to (144.0, 120.2)
- moved R20 2.16 mm to (143.0, 120.2)
- moved U2 2.07 mm to (127.5, 80.8), turned to 0 degrees
- moved Q1 1.00 mm to (141.4, 86.0)
Connections:
- J3 pad 10: /xPB5 -> GND
- J3 pad 11: unconnected-(J3-Pin_11-Pad11) -> /MISC_RX
- J3 pad 12: /ICE_CDONE -> GND
- J3 pad 13: unconnected-(J3-Pin_13-Pad13) -> /CIPO
- J3 pad 14: unconnected-(J3-Pin_14-Pad14) -> GND
- J3 pad 15: GND -> /xPB5
- J3 pad 16: unconnected-(J3-Pin_16-Pad16) -> GND
- J3 pad 17: GND -> unconnected-(J3-Pin_17-Pad17)
- J3 pad 18: unconnected-(J3-Pin_18-Pad18) -> GND
- J3 pad 19: GND -> unconnected-(J3-Pin_19-Pad19)
- J3 pad 2: /CS -> unconnected-(J3-Pin_2-Pad2)
- J3 pad 20: unconnected-(J3-Pin_20-Pad20) -> GND
- J3 pad 3: GND -> /xPB4
- J3 pad 4: /CLK -> GND
- J3 pad 5: GND -> /COPI
- J3 pad 6: /CIPO -> GND
- J3 pad 7: unconnected-(J3-Pin_7-Pad7) -> /CS
- J3 pad 8: /COPI -> GND
- J3 pad 9: /xPB4 -> /CLK
- J8 pad 2: /ICE_CDONE -> /MISC_RX
- RN8 pad 2: /ICE_CDONE -> /MISC_RX
- U6 pad 16: /ICE_CDONE -> /MISC_RX
Routing:
- net /MISC_RX: track 0.00 -> 27.9 mm, vias 0 -> 3
- net /ICE_CDONE: track 27.5 -> 0.00 mm, vias 2 -> 0
- net /CS: track 145.1 -> 132.1 mm, vias 4 -> 2
- net /CLK: track 108.8 -> 97.6 mm, vias 3 -> 5
- net /xPB4: track 55.4 -> 63.4 mm, vias 1 -> 2
- net /CIPO: track 122.6 -> 114.9 mm
- net +1V8: track 11.8 -> 4.18 mm
- net GND: track 51.0 -> 58.5 mm, vias 234 -> 231
- net /xPB5: track 99.1 -> 91.6 mm, vias 0 -> 1
- net VREF: track 120.7 -> 115.7 mm
- net /COPI: track 95.0 -> 91.4 mm, vias 2 -> 1
- net VTARGET: track 167.2 -> 170.4 mm
- net Net-(J5-Pin_4): track 6.04 -> 8.76 mm
- net Net-(J5-Pin_5): track 2.89 -> 5.05 mm
- net /DI: track 89.5 -> 91.1 mm
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Other:
- board text added: "<-JTAG SWD->"
- board text added: "CIPO"
- board text added: "CIPO=MISO=TDO"
- board text added: "CLK"
- board text added: "COPI"
- board text added: "COPI=MOSI=TDI"
- board text added: "CS"
- board text added: "CTS"
- board text added: "CTX"
- board text added: "DCD"
- board text added: "DSR"
- board text added: "DTR"
- board text added: "EN"
- board text added: "GND"
- board text added: "I2C"
- board text added: "JTAG"
- board text added: "Logic Analyzer"
- board text added: "RST"
- board text added: "RTCK"
- board text added: "RTS"
- board text added: "RX-A"
- board text added: "RX-C"
- board text added: "RX-D"
- board text added: "SPI"
- board text added: "SRST"
- board text added: "TCK"
- board text added: "TDI"
- board text added: "TDO"
- board text added: "TMS"
- board text added: "TRST"
- board text added: "TX-A"
- board text added: "TX-A-RX"
- board text added: "TX-C"
- board text added: "TX-C-RX"
- board text added: "TX-D"
- board text added: "TX-D-RX"
- board text added: "UART"
- board text added: "VREF"
- board text added: "VTAR"
- board text added: "WP"

Commit message: Prototype Run 1
Cleaned up libraries for easy export/import. Reversed Polarity of J3, added labels and notes to silkscreen layer. Final version for first prototype run.
Other:
- board text added: "HACK"
